File: skydiving-altimeter/_autosave-stm_32.kicad_sch (KiCad schematic)
At the start: 11 parts, among them J1 Conn_ARM_JTAG_SWD_10, J4 10118193-0001LF, U1 STM32F103C8Tx

Commit message: Switched from the bmp to the lps. Added usb port
Parts:
- J4: footprint AMPHENOL_10118193-0001LF -> Micro USB Port:AMPHENOL_10118193-0001LF
Changed lines of the file:
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@@
       (effects (font (size 1.27 1.27)) (justify left))
     )
-    (property "Footprint" "AMPHENOL_10118193-0001LF" (at 220.98 137.16 0)
+    (property "Footprint" "Micro USB Port:AMPHENOL_10118193-0001LF" (at 220.98 137.16 0)
       (effects (font (size 1.27 1.27)) (justify bottom) hide)
     )
