File: skydiving-altimeter/skydiving-altimeter.kicad_pcb (KiCad board)
At the start: 2 copper layers, 26.3 x 45.1 mm, 27 parts, among them J1 Conn_ARM_JTAG_SWD_10, J2 Battery JST Connector, J3 Conn_01x03, U1 STM32F103C8Tx, U2 BMP581, U4 RP400N501A-TR-FE, U5 LDL1117S33R

Commit message: Switched from the bmp to the lps. Added usb port
Parts:
- removed C8: 100nF, Capacitor_SMD:C_0805_2012Metric
- removed R4, R5: 10, Resistor_SMD:R_0402_1005Metric
- added J4: 10118193-0001LF, Micro USB Port:AMPHENOL_10118193-0001LF, F.Cu at (127.6, 113.1)
- U2: value BMP581 -> LPS22HB; footprint BMP581:BMP581 -> Package_LGA:ST_HLGA-10_2x2mm_P0.5mm_LayoutBorder3x2y
- moved C4 3.24 mm to (125.1, 107.3)
- moved U2 2.62 mm to (125.7, 101.6)
- moved C7 2.54 mm to (122.6, 101.0), turned to 180 degrees
Connections:
- C7 pad 1: GND -> +3V3
- C7 pad 2: Net-(U2-VDD) -> GND
- U1 pad 32: unconnected-(U1-PA11-Pad32) -> Net-(J4-D-)
- U1 pad 33: unconnected-(U1-PA12-Pad33) -> Net-(J4-D+)
- U2 pad 1: Net-(U2-SDO) -> +3V3
- U2 pad 10: Net-(U2-VDD) -> +3V3
- U2 pad 5: Net-(U2-SDO) -> GND
Routing:
- net +5V: track 39.1 -> 57.0 mm
- net +3V3: track 126.2 -> 116.1 mm
- net GND: track 26.3 -> 30.2 mm
- net Net-(J4-D-): track 0.00 -> 3.67 mm
- net Net-(J4-D+): track 0.00 -> 3.67 mm
- net /Baro Sensor/SCL: track 14.0 -> 11.7 mm, vias 4 -> 2
- net /Baro Sensor/SDA: track 21.2 -> 22.3 mm
- net /STM_32/SWDIO: track 32.4 -> 31.4 mm

Commit message: Added external resonator to allow usb
Parts:
- added R4: 1M, Resistor_SMD:R_0805_2012Metric, F.Cu at (110.5, 110.5)
- added Y1: Resonator, JGC42-8828A_CSTNE10M0G550000R0:JGC42-8828A_CSTNE10M0G550000R0, F.Cu at (107.3, 111.7)
- moved C2 3.81 mm to (110.5, 114.3)
- moved C6 3.42 mm to (109.2, 117.5)
Connections:
- U1 pad 5: unconnected-(U1-PD0-Pad5) -> Net-(U1-PD0)
- U1 pad 6: unconnected-(U1-PD1-Pad6) -> Net-(U1-PD1)
Routing:
- net Net-(U1-PD1): track 0.00 -> 6.68 mm
- net Net-(U1-PD0): track 0.00 -> 3.31 mm
- net +3V3: track 116.1 -> 119.0 mm
- net Net-(R4-Pad2): track 0.00 -> 2.26 mm
- net Net-(U1-NRST): track 4.30 -> 2.93 mm

Commit message: Generated gerbers. Added version number to back
Other:
- board text added: "V0.9.3"
Changed lines of the file:
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@@
   (gr_circle (center 127.508 119.888) (end 129.258 119.888)
     (stroke (width 0.1) (type solid)) (fill none) (layer "Edge.Cuts"))
+  (gr_text "V0.9.3" (at 129.54 80.645) (layer "B.SilkS")
+    (effects (font (size 1 1) (thickness 0.15)) (justify left bottom mirror))
+  )
   (gr_text "-" (at 114.808 86.868) (layer "F.SilkS")
     (effects (font (size 1.5 1.5) (thickness 0.3)))
