File: skydiving-altimeter/skydiving-altimeter.kicad_pcb (KiCad board)
At the start: 2 copper layers, 26.3 x 45.1 mm, 27 parts, among them J1 Conn_ARM_JTAG_SWD_10, J2 Battery JST Connector, J3 Conn_01x03, J4 10118193-0001LF, U1 STM32F103C8Tx, U2 LPS22HB, U4 RP400N501A-TR-FE, U5 LDL1117S33R, Y1 Resonator

Commit message: Mostly rerouted
Parts:
- removed J4: 10118193-0001LF, Micro USB Port:AMPHENOL_10118193-0001LF
- added D2: SP0503BAHT, Package_TO_SOT_SMD:SOT-143, B.Cu at (123.6, 119.1)
- added D3: LED, Diode_SMD:D_0603_1608Metric, F.Cu at (108.6, 85.1)
- added D4: LED, Diode_SMD:D_0603_1608Metric, F.Cu at (108.6, 87.0)
- added J5: 10118193-0001LF, Micro USB Port:AMPHENOL_10118193-0001LF, F.Cu at (127.8, 111.3)
- added R5: 22.1k, Resistor_SMD:R_0805_2012Metric, B.Cu at (109.2, 115.6)
- added R6: 47.5k, Resistor_SMD:R_0805_2012Metric, B.Cu at (109.2, 118.5)
- added R7: 1k, Resistor_SMD:R_0805_2012Metric, F.Cu at (111.1, 80.6)
- added R8: 1k, Resistor_SMD:R_0805_2012Metric, F.Cu at (111.1, 84.5)
- added R9: 1k, Resistor_SMD:R_0805_2012Metric, B.Cu at (111.8, 107.3)
- added U3: CP2102N-Axx-xQFN24, Package_DFN_QFN:QFN-24-1EP_4x4mm_P0.5mm_EP2.6x2.6mm, B.Cu at (118.8, 118.1)
- added U6: CAT24M01W, Package_SO:SOIC-8_3.9x4.9mm_P1.27mm, B.Cu at (121.3, 93.3)
- added U7: CAT24M01W, Package_SO:SOIC-8_3.9x4.9mm_P1.27mm, B.Cu at (113.0, 93.3)
- moved C4 2.92 mm to (122.7, 105.7)
- moved C6 1.14 mm to (109.2, 116.3)
- moved C2 1.02 mm to (110.5, 113.3)
Connections:
- U1 pad 30: unconnected-(U1-PA9-Pad30) -> /STM_32/M_TX
- U1 pad 31: unconnected-(U1-PA10-Pad31) -> /STM_32/M_RX
- U1 pad 32: Net-(J4-D-) -> unconnected-(U1-PA11-Pad32)
- U1 pad 33: Net-(J4-D+) -> unconnected-(U1-PA12-Pad33)
Routing:
- net /STM_32/SWCLK: track 28.0 -> 75.8 mm
- net Net-(D3-K): track 0.00 -> 47.4 mm, vias 0 -> 3
- net Net-(D4-K): track 0.00 -> 45.6 mm, vias 0 -> 3
- net +3V3: track 119.0 -> 159.7 mm, vias 0 -> 5
- net Net-(J5-VUSB): track 0.00 -> 34.1 mm, vias 0 -> 1
- net Net-(U3-~{RST}): track 0.00 -> 20.7 mm
- net /Baro Sensor/SCL: track 11.7 -> 31.7 mm, vias 2 -> 3
- net Net-(U3-VBUS): track 0.00 -> 17.2 mm
- net /STM_32/SWDIO: track 31.4 -> 45.6 mm
- net Net-(J5-D-): track 0.00 -> 13.3 mm, vias 0 -> 1
- net Net-(J5-SHIELD-PadS1): track 0.00 -> 11.4 mm, vias 0 -> 4
- net /Baro Sensor/SDA: track 22.3 -> 32.9 mm
- net Net-(J5-D+): track 0.00 -> 10.4 mm, vias 0 -> 1
- net GND: track 30.2 -> 37.9 mm, vias 12 -> 16
- net /STM_32/M_TX: track 0.00 -> 6.81 mm, vias 0 -> 1
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Other:
- board text added: "AltimeX V0.9.4"
- board text removed: "V0.9.3"

Commit message: Completed reroute
Routing:
- net GND: track 37.9 -> 53.7 mm, vias 16 -> 21
- net /STM_32/SWCLK: track 75.8 -> 73.2 mm
- net +3V3: track 159.7 -> 161.6 mm
